Commit message: feat: add Sharpa Hand support, universal calibration tool, and complete vector configs
- Add Sharpa Wave hand (5 fingers, 22 DOF) with URDF, XML, meshes, and all configs
- Fix Sharpa thumb link1 mapping (right_thumb_PP → right_thumb_MC)
- Add qpos_mapping for Sharpa in teleop_sim.py
- Add calibrate_scaling.py: universal scaling calibration for all hands and inputs
- Complete vector configs for all 11 hands × 4 input sources (44 total)
- Add virtual tip links to LinkerHand L21 URDF for vector optimizer compatibility
- Tighten Leap Hand AA joint limits in URDF (±60° → ±11°)
- Remove correct_segment_lengths (caused bent finger distortion)
- Set Video depth_scale default to 1.0
- Add realsense/avp/quest3 input support to debug_skeleton.py
- Add sharpa to teleop_sim.py and debug_skeleton.py robot lists
- Remove deprecated calibrate_noitom.py and benchmark_frames.py
- Update README with Sharpa Hand and calibrate_scaling docs

Co-Authored-By: Claude Opus 4.6 (1M context) <noreply@anthropic.com>

File: assets/leap_hand/leap_hand_left.urdf (robot description, URDF)
Before this commit: robot leap_left, 22 links, 21 joints
Joints:
- joint 0: limit lower=-1.047 upper=1.047 effort=0.95 velocity=8.48 -> lower=-0.2 upper=0.2 effort=0.95 velocity=8.48
- joint 4: limit lower=-1.047 upper=1.047 effort=0.95 velocity=8.48 -> lower=-0.2 upper=0.2 effort=0.95 velocity=8.48
- joint 8: limit lower=-1.047 upper=1.047 effort=0.95 velocity=8.48 -> lower=-0.2 upper=0.2 effort=0.95 velocity=8.48

File: assets/leap_hand/leap_hand_right.urdf (robot description, URDF)
Before this commit: robot leap_right, 22 links, 21 joints
Joints:
- joint 0: limit lower=-1.047 upper=1.047 effort=0.95 velocity=8.48 -> lower=-0.2 upper=0.2 effort=0.95 velocity=8.48
- joint 4: limit lower=-1.047 upper=1.047 effort=0.95 velocity=8.48 -> lower=-0.2 upper=0.2 effort=0.95 velocity=8.48
- joint 8: limit lower=-1.047 upper=1.047 effort=0.95 velocity=8.48 -> lower=-0.2 upper=0.2 effort=0.95 velocity=8.48

File: assets/linkerhand_l21/left/linkerhand_l21_left_vis.urdf (robot description, URDF)
Before this commit: robot linkerhand_l21_left, 18 links, 17 joints
Links:
- added link index_tip
- added link middle_tip
- added link pinky_tip
- added link ring_tip
- added link thumb_tip
Joints:
- added joint index_tip_fixed: type fixed, parent index_middle, child index_tip, origin xyz=0 0 0.044 rpy=0 0 0
- added joint middle_tip_fixed: type fixed, parent middle_middle, child middle_tip, origin xyz=0 0 0.044 rpy=0 0 0
- added joint pinky_tip_fixed: type fixed, parent pinky_middle, child pinky_tip, origin xyz=0 0 0.044 rpy=0 0 0
- added joint ring_tip_fixed: type fixed, parent ring_middle, child ring_tip, origin xyz=0 0 0.044 rpy=0 0 0
- added joint thumb_tip_fixed: type fixed, parent thumb_distal, child thumb_tip, origin xyz=0.040 0 0 rpy=0 0 0

File: assets/linkerhand_l21/right/linkerhand_l21_right_vis.urdf (robot description, URDF)
Before this commit: robot linkerhand_l21_right_urdf, 18 links, 17 joints
Links:
- added link index_tip
- added link middle_tip
- added link pinky_tip
- added link ring_tip
- added link thumb_tip
Joints:
- added joint index_tip_fixed: type fixed, parent index_middle, child index_tip, origin xyz=0 0 0.044 rpy=0 0 0
- added joint middle_tip_fixed: type fixed, parent middle_middle, child middle_tip, origin xyz=0 0 0.044 rpy=0 0 0
- added joint pinky_tip_fixed: type fixed, parent pinky_middle, child pinky_tip, origin xyz=0 0 0.044 rpy=0 0 0
- added joint ring_tip_fixed: type fixed, parent ring_middle, child ring_tip, origin xyz=0 0 0.044 rpy=0 0 0
- added joint thumb_tip_fixed: type fixed, parent thumb_distal, child thumb_tip, origin xyz=0.040 0 0 rpy=0 0 0
