Commit message: feat: add rohand support and improve pico4 teleop
Co-Authored-By: Claude <noreply@anthropic.com>

File: assets/rohand/right/rohand_right_vis.urdf (robot description, URDF)
Before this commit: robot rohand_right, 26 links, 25 joints
Joints:
- joint if_distal_link: mimic (none) -> joint=if_proximal_link multiplier=1.138285 offset=-0.034824
- joint lf_distal_link: mimic (none) -> joint=lf_proximal_link multiplier=1.152366 offset=-0.067444
- joint mf_distal_link: mimic (none) -> joint=mf_proximal_link multiplier=1.139937 offset=-0.033724
- joint rf_distal_link: mimic (none) -> joint=rf_proximal_link multiplier=1.134612 offset=-0.033167
- joint th_distal_link: mimic (none) -> joint=th_proximal_link multiplier=1.229686 offset=-0.037509
